Commit message: modifif du code et rajout des fichier .xacro

File: description/camera.xacro (robot description, xacro)
@@ -1,56 +1,66 @@
 <?xml version="1.0"?>
 <robot xmlns:xacro="http://www.ros.org/wiki/xacro">
-  <!-- Le lien de la caméra -->
-  <link name="camera_link">
-    <visual>
+    <!-- Le lien de la caméra -->
+      <!-- STEP 7 - Camera -->
+  <joint type="fixed" name="camera_joint">
+    <origin xyz="0.315 0 0.075" rpy="0 0 0"/>
+    <child link="camera_link"/>
+    <parent link="chassis"/>
+    <axis xyz="0 1 0" />
+  </joint>
+  <link name='camera_link'>
+    <pose>0 0 0 0 0 0</pose>
+    <inertial>
+      <mass value="0.1"/>
+      <origin xyz="0 0 0" rpy="0 0 0"/>
+      <inertia
+          ixx="1e-6" ixy="0" ixz="0"
+          iyy="1e-6" iyz="0"
+          izz="1e-6"
+      />
+    </inertial>
+    <collision name='collision'>
       <origin xyz="0 0 0" rpy="0 0 0"/>
       <geometry>
-        <box size="0.04 0.04 0.04"/>
+        <box size=".03 .03 .03"/>
       </geometry>
-      <material name="blue"/>
-    </visual>
-    <collision>
+    </collision>
+    <visual name='camera_link_visual'>
       <origin xyz="0 0 0" rpy="0 0 0"/>
       <geometry>
-        <box size="0.04 0.04 0.04"/>
+        <box size=".03 .03 .03"/>
       </geometry>
-    </collision>
-    <xacro:inertial_box mass='0.05'  x=' 0.04' y='0.04' z='0.04'>
-      <origin xyz="0 0 0" rpy="0 0 0"/>
-    </xacro:inertial_box>
+    </visual>
   </link>
-  <!-- Joint qui relie la caméra au châssis -->
-  <joint name="camera_joint" type="fixed">
-    <parent link="chassis"/>
-    <child link="camera_link"/>
-    <origin xyz="0.1 0 0.15" rpy="0 0 0"/>
+  <gazebo reference="camera_link">
+    <material>Gazebo/Red</material>
+  </gazebo>
+  <joint type="fixed" name="camera_optical_joint">
+    <origin xyz="0 0 0" rpy="-1.5707 0 -1.5707"/>
+    <child link="camera_link_optical"/>
+    <parent link="camera_link"/>
   </joint>
-  <!-- Plugin Gazebo pour simuler la caméra -->
+  <link name="camera_link_optical">
+  </link>
+    <!-- Plugin Gazebo pour simuler la caméra -->
   <gazebo reference="camera_link">
-    <sensor name="camera_sensor" type="camera">
-      <always_on>true</always_on>
-      <update_rate>30</update_rate>
-      <visualize>true</visualize>
+    <sensor name="wideangle_camera" type="wideanglecamera">
       <camera>
-        <horizontal_fov>1.3962634</horizontal_fov>
+        <horizontal_fov>3.14</horizontal_fov>
         <image>
           <width>640</width>
           <height>480</height>
-          <format>R8G8B8</format>
         </image>
         <clip>
-          <near>0.05</near>
-          <far>50.0</far>
+          <near>0.1</near>
+          <far>15</far>
         </clip>
+        <optical_frame_id>camera_link_optical</optical_frame_id>
+        <camera_info_topic>camera/camera_info</camera_info_topic>
       </camera>
-      <!-- Plugin ROS-Gazebo -->
-      <!-- <plugin name="camera_controller" filename="libgazebo_ros_camera.so">
-        <ros>
-          <namespace>/</namespace>
-          <remapping>image_raw:=/camera/image_raw</remapping>
-          <remapping>camera_info:=/camera/camera_info</remapping>
-        </ros>
-        <frame_name>camera_link</frame_name>
-      </plugin> -->
+      <always_on>1</always_on>
+      <update_rate>20</update_rate>
+      <topic>camera/image</topic>
+      <gz_frame_id>camera_link</gz_frame_id>
     </sensor>
   </gazebo>

File: description/controle_gazebo.xacro (robot description, xacro)
@@ -2,19 +2,36 @@
 <robot xmlns:xacro="http://www.ros.org/wiki/xacro" >
     <gazebo>
-         <plugin
-            filename="libignition-gazebo-diff-drive-system.so"
-            name="ignition::gazebo::systems::DiffDrive">
+         <plugin filename="gz-sim-diff-drive-system" name="gz::sim::systems::DiffDrive">
+            <odom_publisher_frequency>50</odom_publisher_frequency>
             <left_joint>wheel_left_joint</left_joint>
             <right_joint>wheel_right_joint</right_joint>
-            <wheel_separation>0.297</wheel_separation>
-            <wheel_radius>0.05</wheel_radius>
+            <wheel_separation>0.3</wheel_separation>
+            <wheel_diameter>0.1</wheel_diameter>
+            <max_wheel_torque>200</max_wheel_torque>
+            <max_wheel_acceleration>10.0</max_wheel_acceleration>
+            <!-- <max_velocity>3.0</max_velocity>
+            <max_linear_acceleration>1</max_linear_acceleration>
+            <min_linear_acceleration>-1</min_linear_acceleration>
+            <max_angular_acceleration>2</max_angular_acceleration>
+            <min_angular_acceleration>-2</min_angular_acceleration>
+            <max_linear_velocity>0.5</max_linear_velocity>
+            <min_linear_velocity>-0.5</min_linear_velocity>
+            <max_angular_velocity>1</max_angular_velocity>
+            <min_angular_velocity>-1</min_angular_velocity> -->
             <topic>cmd_vel</topic>
-            <max_linear_acceleration>0.5</max_linear_acceleration>
-            <!-- Output -->
+            <publish_odom>true</publish_odom>
+            <publish_odom_tf>true</publish_odom_tf>
+            <publish_wheel_tf>true</publish_wheel_tf>
+            <odom_topic>odom</odom_topic>
             <frame_id>odom</frame_id>
             <child_frame_id>base_link</child_frame_id>
-            <odom_topic>odom</odom_topic>
-            <odom_publisher_frequency>30</odom_publisher_frequency>
             <tf_topic>/tf</tf_topic>
+         </plugin>
+         <plugin
+            filename="gz-sim-joint-state-publisher-system"
+            name="gz::sim::systems::JointStatePublisher">
+            <topic>joint_states</topic>
+            <joint_name>wheel_left_joint</joint_name>
+            <joint_name>wheel_right_joint</joint_name>
          </plugin>
     </gazebo>

File: description/lidar.xacro (robot description, xacro)
@@ -4,5 +4,5 @@
         <parent link="chassis"/>
         <child link="laser_frame"/>
-        <origin xyz="0.25 0 0.22" rpy="0 0 0"/>
+        <origin xyz="0.06 0 0.125" rpy="0 0 0"/>
     </joint>
     <link name="laser_frame">
@@ -10,11 +10,4 @@
             <geometry>
                 <cylinder radius="0.05" length="0.04"/>
-            </geometry>
-            <material name="black"/>
-        </visual>
-        <visual>
-            <origin xyz="0 0 -0.05"/>
-            <geometry>
-                <cylinder radius="0.01" length="0.1"/>
             </geometry>
             <material name="black"/>
@@ -29,33 +22,33 @@
         </xacro:inertial_cylinder>
     </link>
-    <gazebo reference="laser_frame">
-        <sensor name='laser' type='gpu_lidar'>
-            <pose>0 0 0 0 0 0</pose>
-            <topic>scan</topic>
-            <gz_frame_id>laser_frame</gz_frame_id>
-            <update_rate>10</update_rate>
-            <lidar>
-              <scan>
-                <horizontal>
-                  <samples>640</samples>
-                  <resolution>1</resolution>
-                  <min_angle>-1.396263</min_angle>
-                  <max_angle>1.396263</max_angle>
-                </horizontal>
-                <vertical>
-                  <samples>1</samples>
-                  <resolution>1</resolution>
-                  <min_angle>0.0</min_angle>
-                  <max_angle>0.0</max_angle>
-                </vertical>
-              </scan>
-              <range>
-                <min>0.08</min>
-                <max>10</max>
-                <resolution>0.01</resolution>
-              </range>
-            </lidar>
-            <visualize>true</visualize>
-          </sensor>
+     <gazebo reference="laser_frame">
+            <sensor type="gpu_lidar" name="lidar">
+                <pose>0 0 0 0 0 0</pose>
+                <always_on>true</always_on>
+                <visualize>true</visualize>
+                <update_rate>10</update_rate>
+                <lidar>
+                    <scan>
+                        <horizontal>
+                            <samples>360</samples>
+                            <resolution>1</resolution>
+                            <min_angle>-3.14159</min_angle>
+                            <max_angle>3.14159</max_angle>
+                        </horizontal>
+                    </scan>
+                    <range>
+                        <min>0.2</min>
+                        <max>30.0</max>
+                        <resolution>0.01</resolution>
+                    </range>
+                    <noise>
+                        <type>gaussian</type>
+                        <mean>0.0</mean>
+                        <stddev>0.01</stddev>
+                    </noise>
+                </lidar>
+                <topic>scan</topic>
+                <gz_frame_id>laser_frame</gz_frame_id>
+            </sensor>
     </gazebo>
 </robot>

File: description/robot.urdf.xacro (robot description, xacro)
@@ -6,4 +6,6 @@
      <!--Control robot-->
      <xacro:include filename = "controle_gazebo.xacro"/>
-     <!-- <xacro:include filename='camera.xacro' /> -->
+<!-- camera -->
+     <xacro:include filename='camera.xacro' />
+     <xacro:include filename='imu.xacro'/>
 </robot>

File: description/robot.xacro (robot description, xacro)
@@ -30,5 +30,5 @@
                 <box size="${chassis_length} ${chassis_width} ${chassis_height}"/>
             </geometry>
-            <material name="red"/>
+            <material name="white"/>
         </visual>
         <collision>
@@ -47,6 +47,9 @@
         <parent link="base_link"/>
         <child link="chassis"/>
-        <origin xyz="0 0 0" rpy="0 0 0"/>
+        <origin xyz="-0.1 0 0" rpy="0 0 0"/>
     </joint>
+    <gazebo reference="chassis">
+        <material>Gazebo/White</material>
+    </gazebo>
     <!-- Roue gauche -->
     <link name="wheel_left">
@@ -54,22 +57,31 @@
             <origin xyz="0 0 0" rpy="0 0 0"/>
             <geometry>
-                <cylinder length="0.05" radius="0.05"/>
+                <cylinder length="0.04" radius="0.05"/>
             </geometry>
-            <material name="black"/>
+            <material name="blue"/>
         </visual>
         <collision>
             <origin xyz="0 0 0" rpy="0 0 0"/>
             <geometry>
-                <cylinder length="0.05" radius="0.05"/>
+                <cylinder length="0.04" radius="0.05"/>
             </geometry>
         </collision>
-        <xacro:inertial_cylinder mass="0.1" length="0.05" radius="0.05">
+        <xacro:inertial_cylinder mass="0.1" length="0.04" radius="0.05">
             <origin xyz="0 0 0" rpy="0 0 0"/>
         </xacro:inertial_cylinder>
     </link>
+    <gazebo reference="wheel_left">
+        <material>Gazebo/Blue</material>
+        <mu1>0.2</mu1>
+        <mu2>0.2</mu2>
+        <kp>1000000.0</kp>
+        <kd>100.0</kd>
+        <minDepth>0.0001</minDepth>
+        <maxVel>1.0</maxVel>
+    </gazebo>
     <joint name="wheel_left_joint" type="continuous">
         <parent link="base_link"/>
         <child link="wheel_left"/>
-        <origin xyz="0 ${chassis_width/2 + 0.03} ${0.05/2}" rpy="1.57 0 0"/>
+        <origin xyz="0 ${chassis_width/2 + 0.03} 0" rpy="-1.57 0 0"/>
         <axis xyz="0 0 1"/>
     </joint>
@@ -79,23 +91,32 @@
             <origin xyz="0 0 0" rpy="0 0 0"/>
             <geometry>
-                <cylinder length="0.05" radius="0.05"/>
+                <cylinder length="0.04" radius="0.05"/>
             </geometry>
-            <material name="black"/>
+            <material name="blue"/>
         </visual>
         <collision>
             <origin xyz="0 0 0" rpy="0 0 0"/>
             <geometry>
-                <cylinder length="0.05" radius="0.05"/>
+                <cylinder length="0.04" radius="0.05"/>
             </geometry>
         </collision>
-        <xacro:inertial_cylinder mass="0.1" length="0.05" radius="0.05">
+        <xacro:inertial_cylinder mass="0.1" length="0.04" radius="0.05">
             <origin xyz="0 0 0" rpy="0 0 0"/>
         </xacro:inertial_cylinder>
     </link>
+    <gazebo reference="wheel_right">
+        <material>Gazebo/Blue</material>
+        <mu1>0.2</mu1>
+        <mu2>0.2</mu2>
+        <kp>1000000.0</kp>
+        <kd>100.0</kd>
+        <minDepth>0.0001</minDepth>
+        <maxVel>1.0</maxVel>
+    </gazebo>
     <joint name="wheel_right_joint" type="continuous">
         <parent link="base_link"/>
         <child link="wheel_right"/>
-        <origin xyz="0 -${chassis_width/2 + 0.03} ${0.05/2}" rpy="-1.57 0 0"/>
-        <axis xyz="0 0 1"/>
+        <origin xyz="0 -${chassis_width/2 + 0.03} 0" rpy="1.57 0 0"/>
+        <axis xyz="0 0 -1"/>
     </joint>
     <!-- Roue folle (caster) -->
@@ -105,5 +126,5 @@
                 <sphere radius="0.05"/>
             </geometry>
-            <origin xyz="0.12 0 0" rpy="0 0 0"/>
+            <origin xyz="0 0 0" rpy="0 0 0"/>
             <material name="black"/>
         </visual>
@@ -112,5 +133,5 @@
                 <sphere radius="0.05"/>
             </geometry>
-            <origin xyz="0.12 0 0" rpy="0 0 0"/>
+            <origin xyz="0 0 0" rpy="0 0 0"/>
             <material name="black"/>
         </collision>
@@ -120,7 +141,12 @@
     </link>
     <joint name="caster_wheel_joint" type="fixed">
-        <parent link="base_link"/>
+        <parent link="chassis"/>
         <child link="caster_wheel"/>
-        <origin xyz="0.12 0 0" rpy="0 0 0"/>
+        <origin xyz="0.24 0 0" rpy="0 0 0"/>
     </joint>
+    <gazebo reference="caster_wheel">
+        <material>Gazebo/Black</material>
+        <mu1 value="0.001"/>
+        <mu2 value="0.001"/>
+    </gazebo>
 </robot>
